Commit message: .

File: table/table_description/urdf/table_block.xacro (robot description, xacro)
@@ -5,5 +5,5 @@
 <xacro:property name="M_PI"  value="3.1415"/>
 <joint name="block_joint" type="fixed">
-	<origin xyz="0.15 0.1 ${table_w * 0.5}" rpy="0 0 ${M_PI/2}" />
+	<origin xyz="-0.2 0.15 ${table_w * 0.5}" rpy="0 0 ${M_PI/2}" />
 	<parent link="table_link" />
 	<child link="block_link" />
